File: pcb_layout/Clock2.brd (EAGLE design)
At the start: 100 x 80 mm, 64 parts, among them IC1 7805TV, IC2 74AC138D, Q1 MOSFET-NCHANNELBSS138, Q2 MOSFET-NCHANNELBSS138, Q3 MOSFET-NCHANNELBSS138, Q4 MOSFET-NCHANNELBSS138, Q5 16M, U1 ATMEGA328P_PDIP

Commit message: Updated packages
Parts:
- C1, C2, C3, C4, C5: device rcl:C025-024X044 -> rcl:C1206
- LED1, LED10, LED11, LED12, LED13, LED14, LED15, LED16, LED17, LED18, LED19, LED2, LED20, LED3, LED4, LED5, LED6, LED7, LED8, LED9: device led:1206 -> led:LED3MM
- R1, R10, R11, R12, R13, R14, R15, R16, R17, R18, R19, R1B, R1B1, R1B2, R2, R20, R2B, R3, R3B, R4, R4B, R5, R6, R7, R8, R9, RVCC: device rcl:M3516 -> rcl:R1206
Connections:
- net H_ONE: now also LED13.K, LED18.K, LED2.K, LED8.K; no longer LED13.C, LED18.C, LED2.C, LED8.C
- net H_TEN: now also LED1.K, LED7.K; no longer LED1.C, LED7.C
- net MIN_ONE: now also LED10.K, LED15.K, LED19.K, LED4.K; no longer LED10.C, LED15.C, LED19.C, LED4.C
- net MIN_TEN: now also LED14.K, LED3.K, LED9.K; no longer LED14.C, LED3.C, LED9.C
- net SEC_ONE: now also LED12.K, LED17.K, LED20.K, LED6.K; no longer LED12.C, LED17.C, LED20.C, LED6.C
- net SEC_TEN: now also LED11.K, LED16.K, LED5.K; no longer LED11.C, LED16.C, LED5.C
Routing:
- net N$22: track 85.0 -> 85.8 mm
- net N$10: track 85.0 -> 85.8 mm
- net N$32: track 70.0 -> 70.6 mm
- net H_ONE: track 90.1 -> 90.6 mm
- net MIN_ONE: track 97.5 -> 98.0 mm
- net SEC_ONE: track 118.8 -> 119.3 mm
