File: pcb_layout/Clock2.sch (EAGLE design)
At the start: 64 parts, among them IC1 7805TV, IC2 74AC138D, Q1 MOSFET-NCHANNELBSS138, Q2 MOSFET-NCHANNELBSS138, Q3 MOSFET-NCHANNELBSS138, Q4 MOSFET-NCHANNELBSS138, Q5 16M, U1 ATMEGA328P_PDIP

Commit message: Updated packages
Parts:
- C1, C2, C3, C4, C5: device rcl:C-EU025-024X044 -> rcl:C-EUC1206
- LED1, LED10, LED11, LED12, LED13, LED14, LED15, LED16, LED17, LED18, LED19, LED2, LED20, LED3, LED4, LED5, LED6, LED7, LED8, LED9: device led:LEDSMT1206 -> led:LED3MM
- R1, R10, R11, R12, R13, R14, R15, R16, R17, R18, R19, R1B, R1B1, R1B2, R2, R20, R2B, R3, R3B, R4, R4B, R5, R6, R7, R8, R9, RVCC: device rcl:R-US_M3516 -> rcl:R-US_R1206
Changed lines of the file:
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@@
 <part name="FRAME1" library="frames" deviceset="FRAME_B_L" device=""/>
 <part name="IC1" library="linear" deviceset="78*" device="TV" technology="05" value="7805TV"/>
-<part name="C1" library="rcl" deviceset="C-EU" device="025-024X044" value="33u"/>
-<part name="C2" library="rcl" deviceset="C-EU" device="025-024X044" value="10u"/>
+<part name="C1" library="rcl" deviceset="C-EU" device="C1206" value="33u"/>
+<part name="C2" library="rcl" deviceset="C-EU" device="C1206" value="10u"/>
 <part name="GND1" library="supply1" deviceset="GND" device=""/>
 <part name="U1" library="SparkFun-DigitalIC" deviceset="ATMEGA328P_PDIP" device=""/>
-<part name="RVCC" library="rcl" deviceset="R-US_" device="M3516" value="10k"/>
+<part name="RVCC" library="rcl" deviceset="R-US_" device="R1206" value="10k"/>
 <part name="GND3" library="supply1" deviceset="GND" device=""/>
 <part name="P+3" library="supply1" deviceset="+5V" device=""/>
@@
 <part name="GND4" library="supply1" deviceset="GND" device=""/>
 <part name="Q1" library="SparkFun-DiscreteSemi" deviceset="MOSFET-NCHANNEL" device="BSS138"/>
-<part name="R1" library="rcl" deviceset="R-US_" device="M3516" value="150"/>
-<part name="R1B" library="rcl" deviceset="R-US_" device="M3516" value="4.7k"/>
-<part name="LED1" library="led" deviceset="LED" device="SMT1206"/>
+<part name="R1" library="rcl" deviceset="R-US_" device="R1206" value="150"/>
+<part name="R1B" library="rcl" deviceset="R-US_" device="R1206" value="4.7k"/>
+<part name="LED1" library="led" deviceset="LED" device="3MM"/>
 <part name="IC2" library="74xx-eu" deviceset="74*138" device="D" technology="AC"/>
-<part name="R2" library="rcl" deviceset="R-US_" device="M3516" value="150"/>
-<part name="LED2" library="led" deviceset="LED" device="SMT1206"/>
-<part name="R3" library="rcl" deviceset="R-US_" device="M3516" value="150"/>
-<part name="LED3" library="led" deviceset="LED" device="SMT1206"/>
+<part name="R2" library="rcl" deviceset="R-US_" device="R1206" value="150"/>
+<part name="LED2" library="led" deviceset="LED" device="3MM"/>
+<part name="R3" library="rcl" deviceset="R-US_" device="R1206" value="150"/>
+<part name="LED3" library="led" deviceset="LED" device="3MM"/>
 <part name="Q2" library="SparkFun-DiscreteSemi" deviceset="MOSFET-NCHANNEL" device="BSS138"/>
-<part name="R7" library="rcl" deviceset="R-US_" device="M3516" value="150"/>
-<part name="R2B" library="rcl" deviceset="R-US_" device="M3516" value="4.7k"/>
-<part name="LED7" library="led" deviceset="LED" device="SMT1206"/>
-<part name="R8" library="rcl" deviceset="R-US_" device="M3516" value="150"/>
-<part name="LED8" library="led" deviceset="LED" device="SMT1206"/>
-<part name="R9" library="rcl" deviceset="R-US_" device="M3516" value="150"/>
-<part name="LED9" library="led" deviceset="LED" device="SMT1206"/>
-<part name="R4" library="rcl" deviceset="R-US_" device="M3516" value="150"/>
-<part name="LED4" library="led" deviceset="LED" device="SMT1206"/>
-<part name="R5" library="rcl" deviceset="R-US_" device="M3516" value="150"/>
-<part name="LED5" library="led" deviceset="LED" device="SMT1206"/>
-<part name="R6" library="rcl" deviceset="R-US_" device="M3516" value="150"/>
-<part name="LED6" library="led" deviceset="LED" device="SMT1206"/>
-<part name="R10" library="rcl" deviceset="R-US_" device="M3516" value="150"/>
-<part name="LED10" library="led" deviceset="LED" device="SMT1206"/>
-<part name="R11" library="rcl" deviceset="R-US_" device="M3516" value="150"/>
-<part name="LED11" library="led" deviceset="LED" device="SMT1206"/>
-<part name="R12" library="rcl" deviceset="R-US_" device="M3516" value="150"/>
-<part name="LED12" library="led" deviceset="LED" device="SMT1206"/>
+<part name="R7" library="rcl" deviceset="R-US_" device="R1206" value="150"/>
+<part name="R2B" library="rcl" deviceset="R-US_" device="R1206" value="4.7k"/>
+<part name="LED7" library="led" deviceset="LED" device="3MM"/>
+<part name="R8" library="rcl" deviceset="R-US_" device="R1206" value="150"/>
+<part name="LED8" library="led" deviceset="LED" device="3MM"/>
+<part name="R9" library="rcl" deviceset="R-US_" device="R1206" value="150"/>
+<part name="LED9" library="led" deviceset="LED" device="3MM"/>
+<part name="R4" library="rcl" deviceset="R-US_" device="R1206" value="150"/>
+<part name="LED4" library="led" deviceset="LED" device="3MM"/>
+<part name="R5" library="rcl" deviceset="R-US_" device="R1206" value="150"/>
+<part name="LED5" library="led" deviceset="LED" device="3MM"/>
+<part name="R6" library="rcl" deviceset="R-US_" device="R1206" value="150"/>
+<part name="LED6" library="led" deviceset="LED" device="3MM"/>
+<part name="R10" library="rcl" deviceset="R-US_" device="R1206" value="150"/>
+<part name="LED10" library="led" deviceset="LED" device="3MM"/>
+<part name="R11" library="rcl" deviceset="R-US_" device="R1206" value="150"/>
+<part name="LED11" library="led" deviceset="LED" device="3MM"/>
+<part name="R12" library="rcl" deviceset="R-US_" device="R1206" value="150"/>
+<part name="LED12" library="led" deviceset="LED" device="3MM"/>
 <part name="Q3" library="SparkFun-DiscreteSemi" deviceset="MOSFET-NCHANNEL" device="BSS138"/>
-<part name="R13" library="rcl" deviceset="R-US_" device="M3516" value="150"/>
-<part name="R3B" library="rcl" deviceset="R-US_" device="M3516" value="4.7k"/>
-<part name="LED13" library="led" deviceset="LED" device="SMT1206"/>
+<part name="R13" library="rcl" deviceset="R-US_" device="R1206" value="150"/>
+<part name="R3B" library="rcl" deviceset="R-US_" device="R1206" value="4.7k"/>
+<part name="LED13" library="led" deviceset="LED" device="3MM"/>
 <part name="Q4" library="SparkFun-DiscreteSemi" deviceset="MOSFET-NCHANNEL" device="BSS138"/>
-<part name="R18" library="rcl" deviceset="R-US_" device="M3516" value="150"/>
-<part name="R4B" library="rcl" deviceset="R-US_" device="M3516" value="4.7k"/>
-<part name="LED18" library="led" deviceset="LED" device="SMT1206"/>
-<part name="R14" library="rcl" deviceset="R-US_" device="M3516" value="150"/>
-<part name="LED14" library="led" deviceset="LED" device="SMT1206"/>
-<part name="R15" library="rcl" deviceset="R-US_" device="M3516" value="150"/>
-<part name="LED15" library="led" deviceset="LED" device="SMT1206"/>
-<part name="R19" library="rcl" deviceset="R-US_" device="M3516" value="150"/>
-<part name="LED19" library="led" deviceset="LED" device="SMT1206"/>
-<part name="R16" library="rcl" deviceset="R-US_" device="M3516" value="150"/>
-<part name="LED16" library="led" deviceset="LED" device="SMT1206"/>
-<part name="R17" library="rcl" deviceset="R-US_" device="M3516" value="150"/>
-<part name="LED17" library="led" deviceset="LED" device="SMT1206"/>
-<part name="R20" library="rcl" deviceset="R-US_" device="M3516" value="150"/>
-<part name="LED20" library="led" deviceset="LED" device="SMT1206"/>
+<part name="R18" library="rcl" deviceset="R-US_" device="R1206" value="150"/>
+<part name="R4B" library="rcl" deviceset="R-US_" device="R1206" value="4.7k"/>
+<part name="LED18" library="led" deviceset="LED" device="3MM"/>
+<part name="R14" library="rcl" deviceset="R-US_" device="R1206" value="150"/>
+<part name="LED14" library="led" deviceset="LED" device="3MM"/>
+<part name="R15" library="rcl" deviceset="R-US_" device="R1206" value="150"/>
+<part name="LED15" library="led" deviceset="LED" device="3MM"/>
+<part name="R19" library="rcl" deviceset="R-US_" device="R1206" value="150"/>
+<part name="LED19" library="led" deviceset="LED" device="3MM"/>
+<part name="R16" library="rcl" deviceset="R-US_" device="R1206" value="150"/>
+<part name="LED16" library="led" deviceset="LED" device="3MM"/>
+<part name="R17" library="rcl" deviceset="R-US_" device="R1206" value="150"/>
+<part name="LED17" library="led" deviceset="LED" device="3MM"/>
+<part name="R20" library="rcl" deviceset="R-US_" device="R1206" value="150"/>
+<part name="LED20" library="led" deviceset="LED" device="3MM"/>
 <part name="P+1" library="supply1" deviceset="+5V" device=""/>
 <part name="P+4" library="supply1" deviceset="+5V" device=""/>
@@
 <part name="S1" library="SparkFun-Electromechanical" deviceset="TAC_SWITCH" device="SMD" value="TAC_SWITCHSMD"/>
 <part name="S2" library="SparkFun-Electromechanical" deviceset="TAC_SWITCH" device="SMD" value="TAC_SWITCHSMD"/>
-<part name="R1B1" library="rcl" deviceset="R-US_" device="M3516" value="4.7k"/>
-<part name="R1B2" library="rcl" deviceset="R-US_" device="M3516" value="4.7k"/>
+<part name="R1B1" library="rcl" deviceset="R-US_" device="R1206" value="4.7k"/>
+<part name="R1B2" library="rcl" deviceset="R-US_" device="R1206" value="4.7k"/>
 <part name="GND7" library="supply1" deviceset="GND" device=""/>
 <part name="GND8" library="supply1" deviceset="GND" device=""/>
@@
 <part name="P+5" library="supply1" deviceset="+5V" device=""/>
 <part name="JP2" library="SparkFun-Connectors" deviceset="FTDI_BASIC" device="PTH"/>
-<part name="C3" library="rcl" deviceset="C-EU" device="025-024X044" value="10u"/>
+<part name="C3" library="rcl" deviceset="C-EU" device="C1206" value="10u"/>
 <part name="GND13" library="supply1" deviceset="GND" device=""/>
 <part name="Q5" library="special" deviceset="XTAL/S" device="" value="16M"/>
-<part name="C4" library="rcl" deviceset="C-EU" device="025-024X044" value="18p"/>
-<part name="C5" library="rcl" deviceset="C-EU" device="025-024X044" value="18p"/>
+<part name="C4" library="rcl" deviceset="C-EU" device="C1206" value="18p"/>
+<part name="C5" library="rcl" deviceset="C-EU" device="C1206" value="18p"/>
 </parts>
 <sheets>
