File: pcb_layout/surfacemount/Rev2/Clock2Smaller.brd (EAGLE design)
At the start: 66 x 66 mm, 66 parts, among them IC2 74AC138D, Q1 MOSFET-NCHANNELBSS138, Q2 MOSFET-NCHANNELBSS138, Q3 MOSFET-NCHANNELBSS138, Q4 MOSFET-NCHANNELBSS138, U2 ATMEGA328P_TQFP, X1 CRYSTAL-3.2-2.5

Commit message: board update
Parts:
- C1, C2, C3, C4, C5: device rcl:C1206 -> rcl:C0805
- LED1, LED10, LED11, LED12, LED13, LED14, LED15, LED16, LED17, LED18, LED19, LED2, LED20, LED3, LED4, LED5, LED6, LED7, LED8, LED9: device led:SML1206 -> led:SML0805
- R1, R10, R11, R12, R13, R14, R15, R16, R17, R18, R19, R1B, R1B1, R1B2, R2, R20, R2B, R3, R3B, R4, R4B, R5, R6, R7, R8, R9, RVCC, RVCC1, RVCC2: device rcl:R1206 -> rcl:R0805
- moved C2 38.8 mm to (-20.3, 49.5)
- moved C3 30.0 mm to (-25.4, 49.5)
- moved Q4 25.1 mm to (31.8, 37.5)
- moved R18 25.0 mm to (40.6, 38.1), flipped to the bottom, turned to 90 degrees
- moved R20 23.4 mm to (55.9, 38.1), flipped to the bottom, turned to 90 degrees
- moved R19 23.0 mm to (48.3, 38.1), flipped to the bottom, turned to 90 degrees
- moved JP3 22.6 mm to (8.57, 34.0), flipped to the bottom
- moved R4B 21.2 mm to (31.8, 37.5), flipped to the bottom
- moved Q2 20.8 mm to (31.8, 27.9)
- moved LED18 20.5 mm to (40.6, 38.1), turned to 90 degrees
- moved R13 20.5 mm to (40.6, 33.0), flipped to the bottom, turned to 90 degrees
- moved Q3 19.9 mm to (31.8, 33.0)
- moved RVCC2 19.4 mm to (2.86, 4.13), turned to 270 degrees
- moved R7 18.9 mm to (36.8, 27.9), flipped to the bottom, turned to 90 degrees
- moved R14 18.9 mm to (44.5, 33.0), flipped to the bottom, turned to 90 degrees
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Routing:
- net +5V: track 218.3 -> 36.6 mm, vias 4 -> 3
- net RESET: track 69.3 -> 0.00 mm, vias 2 -> 0
- net MIN_BTN: track 64.6 -> 0.00 mm, vias 2 -> 0
- net HOUR_BTN: track 61.1 -> 0.00 mm, vias 2 -> 0
- net H_ONE: track 87.7 -> 36.5 mm, vias 4 -> 0
- net BIT8: track 54.7 -> 5.45 mm, vias 2 -> 1
- net MIN_ONE: track 80.1 -> 31.4 mm, vias 4 -> 0
- net N$22: track 68.9 -> 23.1 mm, vias 0 -> 1
- net N$10: track 68.9 -> 23.1 mm, vias 0 -> 1
- net BIT2: track 50.6 -> 5.42 mm, vias 2 -> 1
- net MIN_TEN: track 70.4 -> 26.4 mm, vias 3 -> 0
- net SEC_ONE: track 72.6 -> 30.2 mm, vias 4 -> 0
- net SEC_TEN: track 63.4 -> 21.3 mm, vias 3 -> 0
- net BIT4: track 47.3 -> 5.45 mm, vias 2 -> 1
- net H_TEN: track 64.5 -> 23.8 mm, vias 2 -> 0
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Other:
- board size 66 x 66 mm -> 100 x 80 mm
- board text added: "C5"
